File: HW_MFC01/HW_MFC01.kicad_sch (KiCad schematic)
At the start: 78 parts, among them J1 Conn_01x08, J10 Conn_01x04_Pin, J11 Conn_01x02_Pin, J12 Conn_01x02_Pin, J13 Conn_01x02_Pin, J14 Conn_01x02_Pin, J15 Conn_01x08, J18 Conn_01x08, J19 Conn_01x04_Pin, J20 Conn_01x04_Pin, J3 Conn_01x05, J4 Conn_01x07, J5 Conn_01x07, J6 Conn_01x08, J7 Conn_01x06_Pin, J8 Conn_01x02_Pin, J9 Conn_01x02_Pin, Q1 IRLML0030, Q2 IRLML0030, Q3 IRLML0030, Q4 IRLML0030, Q5 IRLML0030, Q6 IRLML0030, Q7 IRLML0030, Q8 IRLML0030, U1 EL3H7, U2 EL3H7, U3 EL3H7, U4 EL3H7, U5 AP63203WU, U6 RP2040-Zero

Commit message: corrected resistor values
Parts:
- R1, R2, R3: value 10k -> 750
- R10, R11, R12, R13, R14, R9: value 10k -> 100
- R4: value 10k -> 470
- R6: value 10k -> 220
Changed lines of the file:
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@@
 	(wire
 		(pts
-			(xy 129.54 163.83) (xy 130.81 163.83)
+			(xy 129.54 163.83) (xy 158.75 163.83)
 		)
 		(stroke
@@
 	(wire
 		(pts
-			(xy 130.81 162.56) (xy 156.21 162.56)
-		)
-		(stroke
-			(width 0)
-			(type default)
-		)
-	)
-	(wire
-		(pts
 			(xy 339.09 60.96) (xy 351.79 60.96)
 		)
@@
 	(wire
 		(pts
-			(xy 130.81 163.83) (xy 130.81 162.56)
-		)
-		(stroke
-			(width 0)
-			(type default)
-		)
-	)
-	(wire
-		(pts
 			(xy 407.67 49.53) (xy 407.67 53.34)
 		)
@@
 	)
 	(label "SBUS_IN"
-		(at 156.21 162.56 180)
+		(at 158.75 163.83 180)
 		(effects
 			(font
@@
 			)
 		)
-		(property "Value" "10k"
+		(property "Value" "750"
 			(at 121.92 77.47 90)
 			(show_name no)
@@
 			)
 		)
-		(property "Value" "10k"
+		(property "Value" "100"
 			(at 351.79 136.906 90)
 			(show_name no)
@@
 			)
 		)
-		(property "Value" "10k"
+		(property "Value" "100"
 			(at 347.98 91.186 90)
 			(show_name no)
@@
 		(in_pos_files yes)
 		(dnp no)
-		(fields_autoplaced yes)
 		(property "Reference" "#FLG03"
 			(at 158.75 167.005 0)
@@
 		)
 		(property "Value" "PWR_FLAG"
-			(at 158.75 163.83 0)
+			(at 165.1 167.64 0)
 			(show_name no)
 			(do_not_autoplace no)
@@
 			)
 		)
-		(property "Value" "10k"
+		(property "Value" "470"
 			(at 121.92 125.73 90)
 			(show_name no)
@@
 			)
 		)
-		(property "Value" "10k"
+		(property "Value" "750"
 			(at 121.92 96.52 90)
 			(show_name no)
@@
 			)
 		)
-		(property "Value" "10k"
+		(property "Value" "100"
 			(at 347.98 86.106 90)
 			(show_name no)
@@
 			)
 		)
-		(property "Value" "10k"
+		(property "Value" "100"
 			(at 351.79 141.986 90)
 			(show_name no)
@@
 			)
 		)
-		(property "Value" "10k"
+		(property "Value" "100"
 			(at 349.25 111.506 90)
 			(show_name no)
@@
 			)
 		)
-		(property "Value" "10k"
+		(property "Value" "750"
 			(at 121.92 50.8 90)
 			(show_name no)
@@
 			)
 		)
-		(property "Value" "10k"
+		(property "Value" "100"
 			(at 349.25 116.586 90)
 			(show_name no)
@@
 			)
 		)
-		(property "Value" "10k"
+		(property "Value" "220"
 			(at 154.94 121.9199 0)
 			(show_name no)

Commit message: updated light sw level values
Parts:
- R7, R8: value 10k -> 43
Changed lines of the file:
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@@
 			)
 		)
-		(property "Value" "10k"
+		(property "Value" "43"
 			(at 335.28 68.326 90)
 			(show_name no)
@@
 			)
 		)
-		(property "Value" "10k"
+		(property "Value" "43"
 			(at 335.28 63.246 90)
 			(show_name no)
